File: KiCad/Sys_ProjectTemplate/Sys_ProjectTemplate.kicad_pcb (KiCad board)
At the start: 2 copper layers, 122 x 84 mm, 7 parts, among them J1 RCA_OUT, J2 RCA_In2, J3 RCA_In1, SW1 SW_Push_DPDT

Commit message: Added Lbls, Description
Other:
- board text added: "RCA In 1"
- board text added: "RCA In 2"
- board text added: "RCA Output"
Changed lines of the file:
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@@
   (general
     (thickness 1.6)
-    (drawings 6)
+    (drawings 9)
     (tracks 0)
     (zones 0)
@@
   )
   (page A4)
+  (title_block
+    (title "Sys Project Template")
+    (date 2020-05-05)
+    (rev 0.0)
+    (company "Philipp Schilk")
+    (comment 1 "No Affiliation with Schiit Audio Products")
+    (comment 2 https://www.schiit.com/products/sys)
+    (comment 3 "For Documentation See: https://github.com/TheSchilk/SYS_ProjectTemplate")
+    (comment 4 "Project Template for a custom PCB fitting the SYS Passive Preamp enclosure.")
+  )
   (layers
     (0 F.Cu signal)
@@
       (net 26 "Net-(SW1-Pad6)"))
   )
+  (gr_text "RCA In 1" (at 180.5 57.75) (layer F.Fab)
+    (effects (font (size 1 1) (thickness 0.15)))
+  )
+  (gr_text "RCA In 2" (at 148.75 57.75) (layer F.Fab)
+    (effects (font (size 1 1) (thickness 0.15)))
+  )
+  (gr_text "RCA Output" (at 97.5 59) (layer F.Fab)
+    (effects (font (size 1 1) (thickness 0.15)))
+  )
   (dimension 84 (width 0.15) (layer Dwgs.User)
